File: loom/loom.kicad_sch (KiCad schematic)
At the start: 0 parts

Commit message: dsfshdagfuwuhgf
Parts:
- added BT1, BT2: Battery_Cell, symbol Device:Battery_Cell
Connections:
- new net: BT1.2 (-), BT2.1 (+)
Other:
- note added: "break light"
- note removed: "battery"
